File: kicad/kb.sch (KiCad schematic (older format))
At the start: 208 parts, among them J1 CHERRY-MX, K1 CHERRY-MX, M1 CHERRY-MX, P1 CHERRY-MX, Q1 CHERRY-MX, T1 CHERRY-MX, T3_2 TEENSY_3.1-3.2_OUTER_ROW, U1 CHERRY-MX, X1 CHERRY-MX, Y1 CHERRY-MX

Commit message: routing done
Parts:
- removed T3_2: TEENSY_3.1-3.2_OUTER_ROW, kicad:TEENSY_3_AND_LC_SERIES_BOARDS_V1.4_TEENSY_3.0-3.2&LC_OUTER_ROW, symbol kb:TEENSY_3_AND_LC_SERIES_BOARDS_V1.4_TEENSY_3.1-3.2_OUTER_ROW
- added T32: TEENSY_3.1-3.2_DIL, Teensy3andLCBoards1_4:TEENSY_3.0-3.2&LC_DIL, symbol Teensy_3_and_LC_Series_Boards_v1.4:TEENSY_3.1-3.2_DIL
- renumbered D95 to G1
