File: kicad/kb.kicad_pcb (KiCad board)
At the start: 2 copper layers, 365.8 x 117.9 mm, 221 parts, among them J1 CHERRY-MX, K1 CHERRY-MX, M1 CHERRY-MX, P1 CHERRY-MX, Q1 CHERRY-MX, T1 CHERRY-MX, T3_2 TEENSY_3.1-3.2_OUTER_ROW, U1 CHERRY-MX, X1 CHERRY-MX, Y1 CHERRY-MX

Commit message: more routing
Routing:
- net /ROW5: track 20.5 -> 559.1 mm, vias 0 -> 5
- net /ROW3: track 21.5 -> 460.7 mm
- net /ROW2: track 20.9 -> 458.1 mm, vias 0 -> 1
- net /ROW4: track 23.0 -> 420.7 mm
- net /ROW6: track 19.5 -> 390.4 mm, vias 0 -> 2
- net /COL0: track 0.00 -> 154.3 mm, vias 0 -> 1
- net /COL3: track 0.00 -> 65.7 mm, vias 0 -> 1
- net /ROW1: track 361.3 -> 407.6 mm, vias 0 -> 1
- net /ROW0: track 355.3 -> 382.6 mm
- net /N$84: track 0.00 -> 14.7 mm
- net /N$61: track 0.00 -> 14.3 mm
- net /N$90: track 0.00 -> 13.9 mm
- net /N$85: track 0.00 -> 13.7 mm
- net /N$89: track 0.00 -> 13.3 mm
- net /COL8: track 0.00 -> 9.42 mm, vias 0 -> 1
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
Commit message: routing done
Parts:
- removed T3_2: TEENSY_3.1-3.2_OUTER_ROW, kicad:TEENSY_3_AND_LC_SERIES_BOARDS_V1.4_TEENSY_3.0-3.2&LC_OUTER_ROW
- added T32: TEENSY_3.1-3.2_DIL, Teensy3andLCBoards1_4:TEENSY_3.0-3.2&LC_DIL, F.Cu at (298.2, -43.7)
- moved TPCOL12 4.56 mm to (260.2, -20.0)
- moved TPROW1 2.83 mm to (-29.0, -18.2)
- moved REF** 1.75 mm to (305.1, -42.1)
- moved REF** 1.52 mm to (255.8, -42.2)
- moved REF** 1.04 mm to (273.6, 43.8)
- moved TPROW0 0.68 mm to (-47.5, -35.8)
- renumbered D95 to G1
Routing:
- net /COL1: track 7.89 -> 500.1 mm, vias 1 -> 3
- net /COL2: track 7.47 -> 473.1 mm, vias 1 -> 3
- net /COL3: track 65.7 -> 521.1 mm, vias 1 -> 3
- net /COL4: track 8.48 -> 412.7 mm, vias 1 -> 9
- net /COL5: track 9.10 -> 402.6 mm, vias 1 -> 3
- net /COL0: track 154.3 -> 542.6 mm, vias 1 -> 7
- net /COL6: track 8.86 -> 333.2 mm, vias 1 -> 3
- net /COL9: track 7.89 -> 313.2 mm, vias 1 -> 7
- net /COL8: track 9.42 -> 295.4 mm, vias 1 -> 3
- net /COL7: track 7.74 -> 288.4 mm, vias 1 -> 4
- net /COL10: track 8.57 -> 267.3 mm, vias 1 -> 3
- net /COL11: track 7.57 -> 259.2 mm, vias 1 -> 7
- net /COL13: track 7.62 -> 197.3 mm, vias 1 -> 3
- net /COL12: track 7.57 -> 170.5 mm
- net /ROW6: track 390.4 -> 481.1 mm, vias 2 -> 4
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Other:
- board size 365.8 x 117.9 mm -> 367.3 x 119.1 mm

Commit message: ready for manuf.
Parts:
- added G***: LOGO, Teensy3andLCBoards1_4:cat, F.Cu at (233.2, -22.8)
- added mnt: MountingHole_2.2mm_M2, MountingHole:MountingHole_2.2mm_M2, F.Cu at (38.0, 5.70)
- added mnt: MountingHole_2.2mm_M2, MountingHole:MountingHole_2.2mm_M2, F.Cu at (127.5, 5.70)
- renumbered REF** to mnt
Routing:
- net /COL3: track 521.1 -> 522.8 mm
Other:
- board text added: "Keyboard Mk.I"
